File: Lattice Solenoid Driver/Lattice Solenoid Driver/Lattice Solenoid Driver.kicad_pcb (KiCad board)
At the start: 2 copper layers, 242.9 x 155.7 mm, 140 parts, among them U1 MCP23017_SS, U15 DRV8873SPWPR, U16 DRV8873SPWPR, U17 DRV8873SPWPR, U18 DRV8873SPWPR, U2 MCP23017_SS, U27 DRV8873SPWPR, U28 DRV8873SPWPR, U29 DRV8873SPWPR, U3 DRV8873SPWPR, U30 DRV8873SPWPR, U39 DRV8873SPWPR, U4 DRV8873SPWPR, U40 DRV8873SPWPR, U41 DRV8873SPWPR, U42 DRV8873SPWPR, U5 DRV8873SPWPR, U6 DRV8873SPWPR

Commit message: Rev1 mostly done
Parts:
- removed U27, U28, U29, U30, U39, U40, U41, U42: DRV8873SPWPR, footprints:PWP24_TEX
- added C115: 1uF, Capacitor_SMD:C_0805_2012Metric, F.Cu at (170.3, 91.5)
- added C116: 100nF, Capacitor_SMD:C_0805_2012Metric, F.Cu at (179.1, 101.8)
- added C117: 47nF, Capacitor_SMD:C_0805_2012Metric, F.Cu at (186.8, 92.4)
- added C118: 100nF, Capacitor_SMD:C_0805_2012Metric, F.Cu at (186.8, 96.9)
- added C119: 1uF, Capacitor_SMD:C_0805_2012Metric, F.Cu at (186.8, 94.7)
- added C120: 10uF, Capacitor_SMD:C_0805_2012Metric, F.Cu at (186.8, 99.4)
- added C121: 10uF, Capacitor_SMD:C_0805_2012Metric, F.Cu at (186.8, 101.8)
- added H1: MountingHole_Pad, MountingHole:MountingHole_3.2mm_M3_DIN965_Pad_TopBottom, F.Cu at (65.2, 103.0)
- added H2: MountingHole_Pad, MountingHole:MountingHole_3.2mm_M3_DIN965_Pad_TopBottom, F.Cu at (65.2, 91.0)
- added H3: MountingHole_Pad, MountingHole:MountingHole_3.2mm_M3_DIN965_Pad_TopBottom, F.Cu at (195.1, 92.0)
- added H4: MountingHole_Pad, MountingHole:MountingHole_3.2mm_M3_DIN965_Pad_TopBottom, F.Cu at (195.1, 102.1)
- added H5: MountingHole_Pad, MountingHole:MountingHole_3.2mm_M3_DIN965_Pad_TopBottom, F.Cu at (198.2, 57.0)
- added H6: MountingHole_Pad, MountingHole:MountingHole_3.2mm_M3_DIN965_Pad_TopBottom, F.Cu at (198.2, 137.0)
- added H7: MountingHole_Pad, MountingHole:MountingHole_3.2mm_M3_DIN965_Pad_TopBottom, F.Cu at (58.1, 137.0)
- added H8: MountingHole_Pad, MountingHole:MountingHole_3.2mm_M3_DIN965_Pad_TopBottom, F.Cu at (58.1, 57.0)
- added J1: Conn_01x06_Pin, Connector_PinHeader_2.54mm:PinHeader_1x06_P2.54mm_Vertical, F.Cu at (75.0, 103.0)
- added J10: Conn_01x05_Pin, Connector_PinHeader_2.54mm:PinHeader_1x05_P2.54mm_Vertical, F.Cu at (165.1, 82.0)
- added J11: Conn_01x05_Pin, Connector_PinHeader_2.54mm:PinHeader_1x05_P2.54mm_Vertical, F.Cu at (182.2, 82.0)
- added J12: Conn_01x05_Pin, Connector_PinHeader_2.54mm:PinHeader_1x05_P2.54mm_Vertical, F.Cu at (192.2, 111.9)
- added J13: Conn_01x05_Pin, Connector_PinHeader_2.54mm:PinHeader_1x05_P2.54mm_Vertical, F.Cu at (175.2, 112.0)
- added J14: Conn_01x05_Pin, Connector_PinHeader_2.54mm:PinHeader_1x05_P2.54mm_Vertical, F.Cu at (158.2, 112.0)
- added J15: Conn_01x05_Pin, Connector_PinHeader_2.54mm:PinHeader_1x05_P2.54mm_Vertical, F.Cu at (141.2, 112.0)
- added J16: Conn_01x05_Pin, Connector_PinHeader_2.54mm:PinHeader_1x05_P2.54mm_Vertical, F.Cu at (124.2, 112.0)
- added J17: Conn_01x05_Pin, Connector_PinHeader_2.54mm:PinHeader_1x05_P2.54mm_Vertical, F.Cu at (107.2, 112.0)
- added J18: Conn_01x05_Pin, Connector_PinHeader_2.54mm:PinHeader_1x05_P2.54mm_Vertical, F.Cu at (90.2, 112.0)
- added J19: Conn_01x05_Pin, Connector_PinHeader_2.54mm:PinHeader_1x05_P2.54mm_Vertical, F.Cu at (73.2, 112.0)
- added J2: Conn_01x02_Pin, Connector_PinHeader_2.54mm:PinHeader_1x02_P2.54mm_Vertical, F.Cu at (69.5, 56.3)
- added J20: Conn_01x02_Pin, Connector_PinHeader_2.54mm:PinHeader_1x02_P2.54mm_Vertical, F.Cu at (103.5, 56.3)
- added J21: Conn_01x02_Pin, Connector_PinHeader_2.54mm:PinHeader_1x02_P2.54mm_Vertical, F.Cu at (120.5, 56.3)
- added J22: Conn_01x02_Pin, Connector_PinHeader_2.54mm:PinHeader_1x02_P2.54mm_Vertical, F.Cu at (137.5, 56.2)
- added J23: Conn_01x02_Pin, Connector_PinHeader_2.54mm:PinHeader_1x02_P2.54mm_Vertical, F.Cu at (154.5, 56.3)
- added J24: Conn_01x02_Pin, Connector_PinHeader_2.54mm:PinHeader_1x02_P2.54mm_Vertical, F.Cu at (171.5, 56.3)
- added J25: Conn_01x02_Pin, Connector_PinHeader_2.54mm:PinHeader_1x02_P2.54mm_Vertical, F.Cu at (188.5, 56.3)
- added J26: Conn_01x02_Pin, Connector_PinHeader_2.54mm:PinHeader_1x02_P2.54mm_Vertical, F.Cu at (185.9, 137.6)
- added J27: Conn_01x02_Pin, Connector_PinHeader_2.54mm:PinHeader_1x02_P2.54mm_Vertical, F.Cu at (168.9, 137.7)
- added J28: Conn_01x02_Pin, Connector_PinHeader_2.54mm:PinHeader_1x02_P2.54mm_Vertical, F.Cu at (151.8, 137.7)
- added J29: Conn_01x02_Pin, Connector_PinHeader_2.54mm:PinHeader_1x02_P2.54mm_Vertical, F.Cu at (134.8, 137.7)
- added J3: Conn_01x05_Pin, Connector_PinHeader_2.54mm:PinHeader_1x05_P2.54mm_Vertical, F.Cu at (63.2, 82.0)
- added J30: Conn_01x02_Pin, Connector_PinHeader_2.54mm:PinHeader_1x02_P2.54mm_Vertical, F.Cu at (117.9, 137.7)
- added J31: Conn_01x02_Pin, Connector_PinHeader_2.54mm:PinHeader_1x02_P2.54mm_Vertical, F.Cu at (100.8, 137.7)
- added J32: Conn_01x02_Pin, Connector_PinHeader_2.54mm:PinHeader_1x02_P2.54mm_Vertical, F.Cu at (83.8, 137.7)
- added J33: Conn_01x02_Pin, Connector_PinHeader_2.54mm:PinHeader_1x02_P2.54mm_Vertical, F.Cu at (66.8, 137.7)
- added J34: Conn_01x05_Pin, Connector_PinHeader_2.54mm:PinHeader_1x05_P2.54mm_Vertical, F.Cu at (166.4, 91.5)
- added J4: Conn_01x05_Pin, Connector_PinHeader_2.54mm:PinHeader_1x05_P2.54mm_Vertical, F.Cu at (80.1, 82.0)
- added J5: Conn_01x02_Pin, Connector_PinHeader_2.54mm:PinHeader_1x02_P2.54mm_Vertical, F.Cu at (86.5, 56.4)
- added J6: Conn_01x05_Pin, Connector_PinHeader_2.54mm:PinHeader_1x05_P2.54mm_Vertical, F.Cu at (97.2, 82.0)
- added J7: Conn_01x05_Pin, Connector_PinHeader_2.54mm:PinHeader_1x05_P2.54mm_Vertical, F.Cu at (114.2, 82.0)
- added J8: Conn_01x05_Pin, Connector_PinHeader_2.54mm:PinHeader_1x05_P2.54mm_Vertical, F.Cu at (131.2, 82.0)
- added J9: Conn_01x05_Pin, Connector_PinHeader_2.54mm:PinHeader_1x05_P2.54mm_Vertical, F.Cu at (148.2, 82.0)
- added U10: DRV8873SPWPR, KiCADv6:PWP24_TEX, F.Cu at (186.7, 71.5)
- added U11: DRV8873SPWPR, KiCADv6:PWP24_TEX, F.Cu at (187.7, 122.4)
- added U12: DRV8873SPWPR, KiCADv6:PWP24_TEX, F.Cu at (170.7, 122.4)
- added U13: DRV8873SPWPR, KiCADv6:PWP24_TEX, F.Cu at (153.7, 122.5)
- added U14: DRV8873SPWPR, KiCADv6:PWP24_TEX, F.Cu at (136.7, 122.5)
- added U19: DRV8873SPWPR, KiCADv6:PWP24_TEX, F.Cu at (176.9, 96.0)
- added U7: DRV8873SPWPR, KiCADv6:PWP24_TEX, F.Cu at (135.7, 71.5)
- added U8: DRV8873SPWPR, KiCADv6:PWP24_TEX, F.Cu at (152.7, 71.5)
- added U9: DRV8873SPWPR, KiCADv6:PWP24_TEX, F.Cu at (169.6, 71.5)
- C10, C101, C17, C35, C38, C45, C63, C66, C7, C73, C91, C94: value 100nF -> 1uF
- C100, C15, C16, C36, C37, C43, C44, C64, C65, C71, C72, C8, C9, C92, C93, C99: value 100nF -> 10uF
- C103, C19, C33, C47, C5, C61, C75, C89: value 1uF -> 47nF
- C104, C20, C32, C34, C4, C48, C6, C60, C62, C76, C88, C90: value 1uF -> 100nF
- C106, C22, C50, C78: value 1uF -> 10uF
- C108, C112, C24, C28, C52, C56, C80, C84: value 10uF -> 1uF
- C109, C111, C25, C27, C53, C55, C81, C83: value 10uF -> 100nF
- C11, C13, C39, C41, C67, C69, C95, C97: value 47nF -> 100nF
- C110, C26, C54, C82: value 10uF -> 47nF
- C14, C42, C70, C98: value 47nF -> 1uF
- U15, U16, U17, U18, U3, U4, U5, U6: footprint footprints:PWP24_TEX -> KiCADv6:PWP24_TEX
- moved JP5 183.9 mm to (82.2, 94.0), turned to 90 degrees
- moved JP2 179.6 mm to (86.2, 94.0), turned to 90 degrees
- moved JP6 176.2 mm to (90.2, 94.0), turned to 90 degrees
- moved U2 149.9 mm to (98.2, 97.0), turned to 180 degrees
- moved U18 149.8 mm to (68.7, 122.5), turned to -90 degrees
- moved C61 149.7 mm to (191.3, 132.3), turned to 90 degrees
- moved C62 144.3 mm to (186.8, 132.2), turned to -90 degrees
- moved C63 144.2 mm to (189.1, 132.2), turned to 90 degrees
- moved C59 144.0 mm to (192.3, 115.7), turned to 180 degrees
- moved C60 139.5 mm to (182.0, 124.5), turned to 90 degrees
- moved C70 139.0 mm to (172.1, 132.3), turned to 90 degrees
- moved C64 138.6 mm to (184.3, 132.2), turned to -90 degrees
- moved U17 138.4 mm to (85.7, 122.5), turned to -90 degrees
- moved C65 134.8 mm to (181.9, 132.2), turned to -90 degrees
- moved C71 133.6 mm to (167.3, 132.3), turned to -90 degrees
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Connections:
- net SOL1+ renamed /H Bridge/SOL+
- net SOL1- renamed /H Bridge/SOL-
- net SOL2+ renamed /H Bridge1/SOL+
- net SOL2- renamed /H Bridge1/SOL-
- net SOL3+ renamed /H Bridge2/SOL+
- net SOL3- renamed /H Bridge2/SOL-
- net SOL4+ renamed /H Bridge3/SOL+
- net SOL4- renamed /H Bridge3/SOL-
- net SOL5+ renamed /H Bridge12/SOL+
- net SOL5- renamed /H Bridge12/SOL-
- net SOL6+ renamed /H Bridge13/SOL+
- net SOL6- renamed /H Bridge13/SOL-
- net SOL7+ renamed /H Bridge14/SOL+
- net SOL7- renamed /H Bridge14/SOL-
- net SOL8+ renamed /H Bridge15/SOL+
- net SOL8- renamed /H Bridge15/SOL-
- C10 pad 1: Net-(U10-30V) -> GND
- C10 pad 2: GND -> VDD
- C100 pad 1: Net-(U48-30V) -> 30V
- C101 pad 1: Net-(U49-30V) -> GND
- C101 pad 2: GND -> VDD
- C102 pad 1: Net-(U50-30V) -> 30V
- C103 pad 1: Net-(U39-VCP) -> Net-(U17-CPL)
- C103 pad 2: Net-(U47-30V) -> Net-(U17-CPH)
- C104 pad 1: Net-(U40-VCP) -> 30V
- C104 pad 2: Net-(U48-30V) -> GND
- C105 pad 1: Net-(U41-VCP) -> Net-(U17-VCP)
- C105 pad 2: Net-(U49-30V) -> 30V
- C106 pad 1: Net-(U42-VCP) -> 30V
- C106 pad 2: Net-(U50-30V) -> GND
- C107 pad 1: Net-(U47-30V) -> 30V
- C108 pad 1: Net-(U48-30V) -> GND
- C108 pad 2: GND -> VDD
- C109 pad 1: Net-(U49-30V) -> 30V
- C11 pad 1: Net-(U3-CPL) -> 30V
- C11 pad 2: Net-(U3-CPH) -> GND
- C110 pad 1: Net-(U50-30V) -> Net-(U18-CPL)
- C110 pad 2: GND -> Net-(U18-CPH)
- C111 pad 1: Net-(U47-30V) -> 30V
- C112 pad 1: Net-(U48-30V) -> Net-(U18-VCP)
- C112 pad 2: GND -> 30V
- C113 pad 1: Net-(U49-30V) -> 30V
- C114 pad 1: Net-(U50-30V) -> 30V
- C13 pad 1: Net-(U5-CPL) -> 30V
- C13 pad 2: Net-(U5-CPH) -> GND
- C14 pad 1: Net-(U6-CPL) -> Net-(U4-VCP)
- C14 pad 2: Net-(U6-CPH) -> 30V
- C15 pad 1: Net-(U11-30V) -> 30V
- C16 pad 1: Net-(U12-30V) -> 30V
- C17 pad 1: Net-(U13-30V) -> GND
- C17 pad 2: GND -> VDD
- C18 pad 1: Net-(U14-30V) -> 30V
- C19 pad 1: Net-(U3-VCP) -> Net-(U5-CPL)
- C19 pad 2: Net-(U11-30V) -> Net-(U5-CPH)
- C20 pad 1: Net-(U4-VCP) -> 30V
- C20 pad 2: Net-(U12-30V) -> GND
- C21 pad 2: Net-(U13-30V) -> 30V
- C22 pad 1: Net-(U6-VCP) -> 30V
- C22 pad 2: Net-(U14-30V) -> GND
- C23 pad 1: Net-(U11-30V) -> 30V
- C24 pad 1: Net-(U12-30V) -> GND
- C24 pad 2: GND -> VDD
- C25 pad 1: Net-(U13-30V) -> 30V
- C26 pad 1: Net-(U14-30V) -> Net-(U6-CPL)
- C26 pad 2: GND -> Net-(U6-CPH)
- C27 pad 1: Net-(U11-30V) -> 30V
- C28 pad 1: Net-(U12-30V) -> Net-(U6-VCP)
- C28 pad 2: GND -> 30V
- C29 pad 1: Net-(U13-30V) -> 30V
- C30 pad 1: Net-(U14-30V) -> 30V
- C32 pad 1: GND -> 30V
- C32 pad 2: VDD -> GND
- C33 pad 1: GND -> Net-(U7-CPL)
- C33 pad 2: VDD -> Net-(U7-CPH)
- C34 pad 1: GND -> 30V
- C34 pad 2: VDD -> GND
- C35 pad 1: Net-(U19-30V) -> Net-(U7-VCP)
- C35 pad 2: GND -> 30V
- C36 pad 1: Net-(U20-30V) -> 30V
- C37 pad 1: Net-(U21-30V) -> 30V
- C38 pad 1: Net-(U22-30V) -> GND
- C38 pad 2: GND -> VDD
- C39 pad 1: Net-(U15-CPL) -> 30V
- C39 pad 2: Net-(U15-CPH) -> GND
- C4 pad 1: GND -> 30V
- C4 pad 2: VDD -> GND
- C40 pad 1: Net-(U16-CPL) -> Net-(U8-CPL)
- C40 pad 2: Net-(U16-CPH) -> Net-(U8-CPH)
- C41 pad 1: Net-(U17-CPL) -> 30V
- C41 pad 2: Net-(U17-CPH) -> GND
- C42 pad 1: Net-(U18-CPL) -> Net-(U8-VCP)
- C42 pad 2: Net-(U18-CPH) -> 30V
- C43 pad 1: Net-(U23-30V) -> 30V
- C44 pad 1: Net-(U24-30V) -> 30V
- C45 pad 1: Net-(U25-30V) -> GND
- C45 pad 2: GND -> VDD
- C46 pad 1: Net-(U26-30V) -> 30V
- C47 pad 1: Net-(U15-VCP) -> Net-(U9-CPL)
- C47 pad 2: Net-(U23-30V) -> Net-(U9-CPH)
- C48 pad 1: Net-(U16-VCP) -> 30V
- C48 pad 2: Net-(U24-30V) -> GND
- C49 pad 1: Net-(U17-VCP) -> Net-(U9-VCP)
- C49 pad 2: Net-(U25-30V) -> 30V
- C5 pad 1: GND -> Net-(U3-CPL)
- C5 pad 2: VDD -> Net-(U3-CPH)
- C50 pad 1: Net-(U18-VCP) -> 30V
- C50 pad 2: Net-(U26-30V) -> GND
- C51 pad 1: Net-(U23-30V) -> 30V
- C52 pad 1: Net-(U24-30V) -> GND
- C52 pad 2: GND -> VDD
- C53 pad 1: Net-(U25-30V) -> 30V
- C54 pad 1: Net-(U26-30V) -> Net-(U10-CPL)
- C54 pad 2: GND -> Net-(U10-CPH)
- C55 pad 1: Net-(U23-30V) -> 30V
- C56 pad 1: Net-(U24-30V) -> Net-(U10-VCP)
- C56 pad 2: GND -> 30V
- C57 pad 1: Net-(U25-30V) -> 30V
- C58 pad 1: Net-(U26-30V) -> 30V
- C6 pad 1: GND -> 30V
- C6 pad 2: VDD -> GND
- C60 pad 1: GND -> 30V
- C60 pad 2: VDD -> GND
- C61 pad 1: GND -> Net-(U11-CPL)
- C61 pad 2: VDD -> Net-(U11-CPH)
- C62 pad 1: GND -> 30V
- C62 pad 2: VDD -> GND
- C63 pad 2: GND -> 30V
- C64 pad 1: Net-(U32-30V) -> 30V
- C65 pad 1: Net-(U33-30V) -> 30V
- C66 pad 1: Net-(U34-30V) -> GND
- C66 pad 2: GND -> VDD
- C67 pad 1: Net-(U27-CPL) -> 30V
- C67 pad 2: Net-(U27-CPH) -> GND
- C69 pad 1: Net-(U29-CPL) -> 30V
- C69 pad 2: Net-(U29-CPH) -> GND
- C7 pad 1: Net-(U7-30V) -> Net-(U3-VCP)
- C7 pad 2: GND -> 30V
- C70 pad 2: Net-(U30-CPH) -> 30V
- C71 pad 1: Net-(U35-30V) -> 30V
- C72 pad 1: Net-(U36-30V) -> 30V
- C73 pad 1: Net-(U37-30V) -> GND
- C73 pad 2: GND -> VDD
- C74 pad 1: Net-(U38-30V) -> 30V
- C75 pad 2: Net-(U35-30V) -> Net-(U13-CPH)
- C76 pad 1: Net-(U28-VCP) -> 30V
- C76 pad 2: Net-(U36-30V) -> GND
- C77 pad 2: Net-(U37-30V) -> 30V
- C78 pad 1: Net-(U30-VCP) -> 30V
- C78 pad 2: Net-(U38-30V) -> GND
- C79 pad 1: Net-(U35-30V) -> 30V
- C8 pad 1: Net-(U8-30V) -> 30V
- C80 pad 1: Net-(U36-30V) -> GND
- C80 pad 2: GND -> VDD
- C81 pad 1: Net-(U37-30V) -> 30V
- C82 pad 1: Net-(U38-30V) -> Net-(U14-CPL)
- C82 pad 2: GND -> Net-(U14-CPH)
- C83 pad 1: Net-(U35-30V) -> 30V
- C84 pad 1: Net-(U36-30V) -> Net-(U14-VCP)
- C84 pad 2: GND -> 30V
- C85 pad 1: Net-(U37-30V) -> 30V
- C86 pad 1: Net-(U38-30V) -> 30V
- C88 pad 1: GND -> 30V
- C88 pad 2: VDD -> GND
- C89 pad 1: GND -> Net-(U15-CPL)
- C89 pad 2: VDD -> Net-(U15-CPH)
- C9 pad 1: Net-(U9-30V) -> 30V
- C90 pad 1: GND -> 30V
- C90 pad 2: VDD -> GND
- C91 pad 1: Net-(U43-30V) -> Net-(U15-VCP)
- C91 pad 2: GND -> 30V
- C92 pad 1: Net-(U44-30V) -> 30V
- C93 pad 1: Net-(U45-30V) -> 30V
- C94 pad 1: Net-(U46-30V) -> GND
- C94 pad 2: GND -> VDD
- C95 pad 1: Net-(U39-CPL) -> 30V
- C95 pad 2: Net-(U39-CPH) -> GND
- C96 pad 1: Net-(U40-CPL) -> Net-(U16-CPL)
- C96 pad 2: Net-(U40-CPH) -> Net-(U16-CPH)
- C97 pad 1: Net-(U41-CPL) -> 30V
- C97 pad 2: Net-(U41-CPH) -> GND
- C98 pad 1: Net-(U42-CPL) -> Net-(U16-VCP)
- C98 pad 2: Net-(U42-CPH) -> 30V
- C99 pad 1: Net-(U47-30V) -> 30V
- U15 pad 11: unconnected-(U15-NSLEEP-Pad11) -> VDD
- U15 pad 13: Net-(U19-30V) -> 30V
- U15 pad 2: unconnected-(U15-NFAULT-Pad2) -> Net-(J16-Pin_1)
- U15 pad 20: Net-(U23-30V) -> 30V
- U15 pad 3: unconnected-(U15-SDO-Pad3) -> Net-(J16-Pin_2)
- U15 pad 4: unconnected-(U15-SDI-Pad4) -> Net-(J16-Pin_3)
- U15 pad 5: unconnected-(U15-SCLK-Pad5) -> Net-(J16-Pin_4)
- U15 pad 6: unconnected-(U15-NSCS-Pad6) -> Net-(J16-Pin_5)
- U15 pad 7: EN5 -> EN13
- U15 pad 8: PH5 -> PH13
- U15 pad 9: unconnected-(U15-DISABLE-Pad9) -> GND
- U16 pad 11: unconnected-(U16-NSLEEP-Pad11) -> VDD
- U16 pad 13: Net-(U20-30V) -> 30V
- U16 pad 2: unconnected-(U16-NFAULT-Pad2) -> Net-(J17-Pin_1)
- U16 pad 20: Net-(U24-30V) -> 30V
- U16 pad 3: unconnected-(U16-SDO-Pad3) -> Net-(J17-Pin_2)
- U16 pad 4: unconnected-(U16-SDI-Pad4) -> Net-(J17-Pin_3)
- U16 pad 5: unconnected-(U16-SCLK-Pad5) -> Net-(J17-Pin_4)
- U16 pad 6: unconnected-(U16-NSCS-Pad6) -> Net-(J17-Pin_5)
- U16 pad 7: EN6 -> EN14
- U16 pad 8: PH6 -> PH14
- U16 pad 9: unconnected-(U16-DISABLE-Pad9) -> GND
- U17 pad 11: unconnected-(U17-NSLEEP-Pad11) -> VDD
- U17 pad 13: Net-(U21-30V) -> 30V
- U17 pad 2: unconnected-(U17-NFAULT-Pad2) -> Net-(J18-Pin_1)
- U17 pad 20: Net-(U25-30V) -> 30V
- U17 pad 3: unconnected-(U17-SDO-Pad3) -> Net-(J18-Pin_2)
- U17 pad 4: unconnected-(U17-SDI-Pad4) -> Net-(J18-Pin_3)
- U17 pad 5: unconnected-(U17-SCLK-Pad5) -> Net-(J18-Pin_4)
- U17 pad 6: unconnected-(U17-NSCS-Pad6) -> Net-(J18-Pin_5)
- U17 pad 7: EN7 -> EN15
- U17 pad 8: PH7 -> PH15
- U17 pad 9: unconnected-(U17-DISABLE-Pad9) -> GND
- U18 pad 11: unconnected-(U18-NSLEEP-Pad11) -> VDD
- U18 pad 13: Net-(U22-30V) -> 30V
- U18 pad 2: unconnected-(U18-NFAULT-Pad2) -> Net-(J19-Pin_1)
- U18 pad 20: Net-(U26-30V) -> 30V
- U18 pad 3: unconnected-(U18-SDO-Pad3) -> Net-(J19-Pin_2)
- U18 pad 4: unconnected-(U18-SDI-Pad4) -> Net-(J19-Pin_3)
- U18 pad 5: unconnected-(U18-SCLK-Pad5) -> Net-(J19-Pin_4)
- U18 pad 6: unconnected-(U18-NSCS-Pad6) -> Net-(J19-Pin_5)
- U18 pad 7: EN8 -> EN16
- U18 pad 8: PH8 -> PH16
- U18 pad 9: unconnected-(U18-DISABLE-Pad9) -> GND
- U3 pad 11: unconnected-(U3-NSLEEP-Pad11) -> VDD
- U3 pad 13: Net-(U7-30V) -> 30V
- U3 pad 2: unconnected-(U3-NFAULT-Pad2) -> Net-(J3-Pin_1)
- U3 pad 20: Net-(U11-30V) -> 30V
- U3 pad 3: unconnected-(U3-SDO-Pad3) -> Net-(J3-Pin_2)
- U3 pad 4: unconnected-(U3-SDI-Pad4) -> Net-(J3-Pin_3)
- U3 pad 5: unconnected-(U3-SCLK-Pad5) -> Net-(J3-Pin_4)
- U3 pad 6: unconnected-(U3-NSCS-Pad6) -> Net-(J3-Pin_5)
- U3 pad 9: unconnected-(U3-DISABLE-Pad9) -> GND
- U4 pad 11: unconnected-(U4-NSLEEP-Pad11) -> VDD
- U4 pad 13: Net-(U8-30V) -> 30V
- U4 pad 2: unconnected-(U4-NFAULT-Pad2) -> Net-(J4-Pin_1)
- U4 pad 20: Net-(U12-30V) -> 30V
- U4 pad 3: unconnected-(U4-SDO-Pad3) -> Net-(J4-Pin_2)
- U4 pad 4: unconnected-(U4-SDI-Pad4) -> Net-(J4-Pin_3)
- U4 pad 5: unconnected-(U4-SCLK-Pad5) -> Net-(J4-Pin_4)
- U4 pad 6: unconnected-(U4-NSCS-Pad6) -> Net-(J4-Pin_5)
- U4 pad 9: unconnected-(U4-DISABLE-Pad9) -> GND
- U5 pad 11: unconnected-(U5-NSLEEP-Pad11) -> VDD
- U5 pad 13: Net-(U9-30V) -> 30V
- U5 pad 2: unconnected-(U5-NFAULT-Pad2) -> Net-(J6-Pin_1)
- U5 pad 20: Net-(U13-30V) -> 30V
- U5 pad 3: unconnected-(U5-SDO-Pad3) -> Net-(J6-Pin_2)
- U5 pad 4: unconnected-(U5-SDI-Pad4) -> Net-(J6-Pin_3)
- U5 pad 5: unconnected-(U5-SCLK-Pad5) -> Net-(J6-Pin_4)
- U5 pad 6: unconnected-(U5-NSCS-Pad6) -> Net-(J6-Pin_5)
- U5 pad 9: unconnected-(U5-DISABLE-Pad9) -> GND
- U6 pad 11: unconnected-(U6-NSLEEP-Pad11) -> VDD
- U6 pad 13: Net-(U10-30V) -> 30V
- U6 pad 2: unconnected-(U6-NFAULT-Pad2) -> Net-(J7-Pin_1)
- U6 pad 20: Net-(U14-30V) -> 30V
- U6 pad 3: unconnected-(U6-SDO-Pad3) -> Net-(J7-Pin_2)
- U6 pad 4: unconnected-(U6-SDI-Pad4) -> Net-(J7-Pin_3)
- U6 pad 5: unconnected-(U6-SCLK-Pad5) -> Net-(J7-Pin_4)
- U6 pad 6: unconnected-(U6-NSCS-Pad6) -> Net-(J7-Pin_5)
- U6 pad 9: unconnected-(U6-DISABLE-Pad9) -> GND
Routing:
- net 30V: track 0.00 -> 947.2 mm, vias 0 -> 51
- net GND: track 0.00 -> 735.1 mm, vias 0 -> 299
- net VDD: track 0.00 -> 229.6 mm, vias 0 -> 16
- net LOAD PH: track 0.00 -> 108.8 mm, vias 0 -> 8
- net LOAD EN: track 0.00 -> 105.3 mm, vias 0 -> 6
- net EN9: track 0.00 -> 95.5 mm
- net PH9: track 0.00 -> 94.6 mm
- net PH10: track 0.00 -> 85.2 mm, vias 0 -> 2
- net EN8: track 0.00 -> 82.5 mm, vias 0 -> 2
- net EN10: track 0.00 -> 80.5 mm, vias 0 -> 2
- net EN1: track 0.00 -> 80.4 mm
- net PH8: track 0.00 -> 80.3 mm, vias 0 -> 2
- net PH1: track 0.00 -> 76.2 mm
- net EN11: track 0.00 -> 75.7 mm, vias 0 -> 2
- net PH11: track 0.00 -> 71.4 mm, vias 0 -> 2
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- added copper zone on B.Cu, net 30V
- added copper zone on F.Cu, net 30V
- added copper zone on B.Cu, net GND
- added copper zone on F.Cu, net GND
- added copper zone on F.Cu, net VDD
Other:
- board size 242.9 x 155.7 mm -> 148 x 88 mm
- board text added: "+ -"
- board text added: "30V"
- board text added: "5V"
- board text added: "A0"
- board text added: "A1"
- board text added: "A2"
- board text added: "EN L"
- board text added: "FAULT"
- board text added: "GND"
- board text added: "LATTICE SOLENOID DRIVER REV. 1 JACOB MUKOBI"
- board text added: "MOT. +"
- board text added: "MOT. -"
- board text added: "NSCS"
- board text added: "PH L"
- board text added: "PWR IN"
- board text added: "SCL"
- board text added: "SCLK"
- board text added: "SDA"
- board text added: "SDI"
- board text added: "SDO"
- board text added: "SOL.1"
- board text added: "SOL.10"
- board text added: "SOL.11"
- board text added: "SOL.12"
- board text added: "SOL.13"
- board text added: "SOL.14"
- board text added: "SOL.15"
- board text added: "SOL.16"
- board text added: "SOL.2"
- board text added: "SOL.3"
- board text added: "SOL.4"
- board text added: "SOL.5"
- board text added: "SOL.6"
- board text added: "SOL.7"
- board text added: "SOL.8"
- board text added: "SOL.9"

Commit message: Finished Rev 1 initial
Parts:
- moved C24 22.2 mm to (136.2, 78.3)
- moved C29 22.2 mm to (144.2, 61.8)
- moved J17 22.2 mm to (129.3, 112.1)
- moved J30 22.2 mm to (140.1, 137.8)
- moved C114 22.2 mm to (85.1, 132.4)
- moved H7 22.2 mm to (80.3, 137.1)
- moved H8 22.2 mm to (80.3, 57.1)
- moved C1 22.2 mm to (147.3, 98.1)
- moved C10 22.2 mm to (102.2, 78.3)
- moved C100 22.2 mm to (119.1, 132.4)
- moved C101 22.2 mm to (112.4, 115.9)
- moved C103 22.2 mm to (111.5, 132.5)
- moved C104 22.2 mm to (107.0, 132.4)
- moved C105 22.2 mm to (109.2, 132.4)
- moved C106 22.2 mm to (104.5, 132.4)
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Connections:
- U10 pad EPAD: (no net) -> GND
- U12 pad EPAD: (no net) -> GND
- U13 pad EPAD: (no net) -> GND
- U14 pad EPAD: (no net) -> GND
- U15 pad EPAD: (no net) -> GND
- U16 pad EPAD: (no net) -> GND
- U17 pad EPAD: (no net) -> GND
- U18 pad EPAD: (no net) -> GND
- U19 pad EPAD: (no net) -> GND
- U3 pad EPAD: (no net) -> GND
- U4 pad EPAD: (no net) -> GND
- U5 pad EPAD: (no net) -> GND
- U6 pad EPAD: (no net) -> GND
- U7 pad EPAD: (no net) -> GND
- U8 pad EPAD: (no net) -> GND
- U9 pad EPAD: (no net) -> GND
Routing:
- net VDD: track 229.6 -> 253.6 mm, vias 16 -> 20
- net Net-(J14-Pin_5): track 22.8 -> 13.1 mm
- net EN7: track 67.9 -> 58.9 mm
- net EN12: track 59.8 -> 50.8 mm
- net EN4: track 42.2 -> 33.2 mm
- net EN5: track 40.8 -> 31.8 mm
- net EN3: track 52.4 -> 43.4 mm
- net EN11: track 75.7 -> 66.7 mm
- net EN2: track 65.8 -> 56.8 mm
- net EN13: track 45.5 -> 36.6 mm
- net EN1: track 80.4 -> 71.4 mm
- net EN6: track 50.2 -> 41.5 mm
- net EN8: track 82.5 -> 74.0 mm
- net EN14: track 35.3 -> 26.9 mm
- net PH12: track 55.8 -> 50.0 mm
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Other:
- board text added: "FLT"
- board text removed: "FAULT"

Commit message: Final Stepper Edits
Parts:
- added AOUT1: MountingHole_Pad, MountingHole:MountingHole_3.2mm_M3_DIN965_Pad_TopBottom, F.Cu at (244.0, 110.5)
- added AOUT2: MountingHole_Pad, MountingHole:MountingHole_3.2mm_M3_DIN965_Pad_TopBottom, F.Cu at (236.0, 110.5)
- added BOUT1: MountingHole_Pad, MountingHole:MountingHole_3.2mm_M3_DIN965_Pad_TopBottom, F.Cu at (220.5, 110.5)
- added BOUT2: MountingHole_Pad, MountingHole:MountingHole_3.2mm_M3_DIN965_Pad_TopBottom, F.Cu at (228.0, 110.5)
- added C122: 10nF, Capacitor_SMD:C_0805_2012Metric, F.Cu at (228.5, 125.1)
- added C123: 100nF, Capacitor_SMD:C_0805_2012Metric, F.Cu at (228.5, 121.6)
- added C124: 100nF, Capacitor_SMD:C_0805_2012Metric, F.Cu at (228.5, 116.6)
- added C125: 470nF, Capacitor_SMD:C_0805_2012Metric, F.Cu at (220.5, 138.0)
- added J35: Conn_01x09_Pin, Connector_PinHeader_2.54mm:PinHeader_1x09_P2.54mm_Vertical, F.Cu at (233.0, 117.0)
- added J36: Conn_01x02_Pin, Connector_PinHeader_2.54mm:PinHeader_1x02_P2.54mm_Vertical, F.Cu at (238.9, 130.0)
- added R3: 1M, Resistor_SMD:R_0805_2012Metric, F.Cu at (228.5, 119.1)
- added R4: 200m, Resistor_SMD:R_0805_2012Metric, F.Cu at (221.0, 119.1)
- added R5: 200m, Resistor_SMD:R_0805_2012Metric, F.Cu at (221.0, 116.6)
- added R6: 50k, Resistor_SMD:R_0805_2012Metric, F.Cu at (221.0, 121.6)
- added R7: 30k, Resistor_SMD:R_0805_2012Metric, F.Cu at (221.0, 124.1)
- added U20: DRV8825PWPR, footprints:PWP28_5P18X3P1, F.Cu at (224.8, 131.1)
- moved H6 23.7 mm to (244.0, 137.0)
- moved H5 23.7 mm to (244.0, 57.1)
- moved H7 0.31 mm to (80.0, 137.1)
- moved H8 0.31 mm to (80.0, 57.1)
Routing:
- net 30V: track 950.9 -> 1027.3 mm, vias 51 -> 54
- net Net-(J35-Pin_3): track 0.00 -> 35.6 mm
- net /Load Stepper Driver/AOUT1: track 0.00 -> 32.7 mm
- net Net-(J35-Pin_4): track 0.00 -> 31.5 mm
- net Net-(J35-Pin_1): track 0.00 -> 30.3 mm, vias 0 -> 1
- net Net-(J35-Pin_5): track 0.00 -> 26.8 mm
- net /Load Stepper Driver/AOUT2: track 0.00 -> 25.5 mm
- net GND: track 737.3 -> 761.7 mm, vias 304 -> 310
- net Net-(J35-Pin_2): track 0.00 -> 23.0 mm, vias 0 -> 1
- net Net-(J35-Pin_6): track 0.00 -> 21.5 mm
- net /Load Stepper Driver/BOUT2: track 0.00 -> 19.6 mm
- net /Load Stepper Driver/DIR: track 0.00 -> 19.5 mm, vias 0 -> 1
- net /Load Stepper Driver/BOUT1: track 0.00 -> 19.0 mm
- net Net-(U20-ISENB): track 0.00 -> 18.2 mm, vias 0 -> 2
- net Net-(J35-Pin_7): track 0.00 -> 17.4 mm
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Other:
- board size 148 x 88 mm -> 172 x 88 mm
- board text added: "DIR"
- board text added: "LATTICE ACTUATOR DRIVER REV. 1, JACOB MUKOBI"
- board text added: "STEP"
- board text removed: "LATTICE SOLENOID DRIVER REV. 1 JACOB MUKOBI"
